File: kicad/yaesu_icom_atu_seq_v2.kicad_pcb (KiCad board)
At the start: 2 copper layers, 160.4 x 158.2 mm, 113 parts, among them J1 ICOM ATU, J10 TXGLINK, J11 PGLINK, J12 POWER, J13 Icom ATU, J14 I2C, J15 ALC OUT, J16 SEQ A1-3, J17 SEQ B1-3, J18 SEQ C1-3, J19 SEQ D1-3, J2 STBY, J3 TUNER, J4 POWER, J5 I2C, J6 ALC, J7 STBY, J8 TUNER, J9 PVLINK, U1 PC817, U10 PC817, U11 PC817, U12 PC817, U13 PC817, U14 PC817, U15 PC817, U16 PC817, U2 L7805, U3 PC817, U4 PC817, U5 PC817, U6 PC817, U7 PC817, U8 PC817, U9 PC817

Commit message: Update schematic and PCB
Parts:
- removed the REF** at (190.5, 127.0) (x2)
- removed the REF** at (120.3, 94.0)
- removed U10, U11, U12, U13, U14, U15, U16, U8, U9: PC817, Custom:PC817_DIP
- added BZ1: Buzzer, Buzzer_Beeper:Buzzer_TDK_PS1240P02BT_D12.2mm_H6.5mm, F.Cu at (100.4, 213.4)
- added C11: 10n, Capacitor_THT:C_Disc_D4.3mm_W1.9mm_P5.00mm, F.Cu at (276.9, 95.2)
- added C12: 10n, Capacitor_THT:C_Disc_D4.3mm_W1.9mm_P5.00mm, F.Cu at (193.0, 124.5)
- added C13: 10n, Capacitor_THT:C_Disc_D4.3mm_W1.9mm_P5.00mm, F.Cu at (189.2, 124.5)
- added C15: 10n, Capacitor_THT:C_Disc_D4.3mm_W1.9mm_P5.00mm, F.Cu at (269.2, 95.2)
- added C19: 100n, Capacitor_THT:C_Disc_D4.3mm_W1.9mm_P5.00mm, F.Cu at (134.4, 74.2)
- added C2: 100n, Capacitor_THT:C_Disc_D4.3mm_W1.9mm_P5.00mm, F.Cu at (139.4, 70.4)
- added C20: 100n, Capacitor_THT:C_Disc_D4.3mm_W1.9mm_P5.00mm, F.Cu at (131.8, 70.4)
- added C24: 100n, Capacitor_THT:C_Disc_D4.3mm_W1.9mm_P5.00mm, F.Cu at (105.5, 191.8)
- added C25: 10nF, Capacitor_THT:C_Disc_D5.1mm_W3.2mm_P5.00mm, F.Cu at (149.9, 222.2)
- added C26: 10nF, Capacitor_THT:C_Disc_D5.1mm_W3.2mm_P5.00mm, F.Cu at (160.0, 222.2)
- added C27: 10nF, Capacitor_THT:C_Disc_D5.1mm_W3.2mm_P5.00mm, F.Cu at (170.2, 222.2)
- added C28: 10nF, Capacitor_THT:C_Disc_D5.1mm_W3.2mm_P5.00mm, F.Cu at (180.3, 222.2)
- added C29: 10nF, Capacitor_THT:C_Disc_D5.1mm_W3.2mm_P5.00mm, F.Cu at (190.5, 222.2)
- added C3: 10n, Capacitor_THT:C_Disc_D4.3mm_W1.9mm_P5.00mm, F.Cu at (189.2, 97.8)
- added C30: 10nF, Capacitor_THT:C_Disc_D5.1mm_W3.2mm_P5.00mm, F.Cu at (200.7, 222.2)
- added C31: 10nF, Capacitor_THT:C_Disc_D5.1mm_W3.2mm_P5.00mm, F.Cu at (219.7, 222.2)
- added C32: 10nF, Capacitor_THT:C_Disc_D5.1mm_W3.2mm_P5.00mm, F.Cu at (229.9, 222.2)
- added C33: 10nF, Capacitor_THT:C_Disc_D5.1mm_W3.2mm_P5.00mm, F.Cu at (240.0, 222.2)
- added C34: 10nF, Capacitor_THT:C_Disc_D5.1mm_W3.2mm_P5.00mm, F.Cu at (250.2, 222.2)
- added C35: 10nF, Capacitor_THT:C_Disc_D5.1mm_W3.2mm_P5.00mm, F.Cu at (260.4, 222.2)
- added C36: 10nF, Capacitor_THT:C_Disc_D5.1mm_W3.2mm_P5.00mm, F.Cu at (270.5, 222.2)
- added C4: 100n, Capacitor_THT:C_Disc_D4.3mm_W1.9mm_P5.00mm, F.Cu at (126.8, 74.2)
- added C6: 100n, Capacitor_THT:C_Disc_D4.3mm_W1.9mm_P5.00mm, F.Cu at (196.6, 62.3)
- added C7: 10n, Capacitor_THT:C_Disc_D4.3mm_W1.9mm_P5.00mm, F.Cu at (185.4, 97.8)
- added C8: 10n, Capacitor_THT:C_Disc_D4.3mm_W1.9mm_P5.00mm, F.Cu at (181.6, 97.8)
- added C9: 10n, Capacitor_THT:C_Disc_D4.3mm_W1.9mm_P5.00mm, F.Cu at (193.0, 102.8)
- added D1: 1.5KE18A, Diode_THT:D_DO-201AE_P15.24mm_Horizontal, F.Cu at (268.0, 67.3)
- added D2: 1.5KE18A, Diode_THT:D_DO-201AE_P15.24mm_Horizontal, F.Cu at (260.4, 67.3)
- added D27: 1N4148, Diode_THT:D_DO-35_SOD27_P7.62mm_Horizontal, F.Cu at (100.3, 203.2)
- added D28: 1.5KE18A, Diode_THT:D_DO-201AE_P15.24mm_Horizontal, F.Cu at (175.3, 221.0)
- added D29: 1.5KE18A, Diode_THT:D_DO-201AE_P15.24mm_Horizontal, F.Cu at (185.4, 221.0)
- added D3: 1N4148, Diode_THT:D_DO-35_SOD27_P7.62mm_Horizontal, F.Cu at (273.1, 100.3)
- added D30: 1.5KE18A, Diode_THT:D_DO-201AE_P15.24mm_Horizontal, F.Cu at (195.6, 221.0)
- added D31: 1.5KE18A, Diode_THT:D_DO-201AE_P15.24mm_Horizontal, F.Cu at (144.8, 221.0)
- added D32: 1.5KE18A, Diode_THT:D_DO-201AE_P15.24mm_Horizontal, F.Cu at (154.9, 221.0)
- added D33: 1.5KE18A, Diode_THT:D_DO-201AE_P15.24mm_Horizontal, F.Cu at (165.1, 221.0)
- added D34: 1.5KE18A, Diode_THT:D_DO-201AE_P15.24mm_Horizontal, F.Cu at (214.6, 221.0)
- added D35: 1.5KE18A, Diode_THT:D_DO-201AE_P15.24mm_Horizontal, F.Cu at (224.8, 221.0)
- added D36: 1.5KE18A, Diode_THT:D_DO-201AE_P15.24mm_Horizontal, F.Cu at (234.9, 221.0)
- added D37: 1.5KE18A, Diode_THT:D_DO-201AE_P15.24mm_Horizontal, F.Cu at (245.1, 221.0)
- added D38: 1.5KE18A, Diode_THT:D_DO-201AE_P15.24mm_Horizontal, F.Cu at (255.3, 221.0)
- added D39: 1.5KE18A, Diode_THT:D_DO-201AE_P15.24mm_Horizontal, F.Cu at (265.4, 221.0)
- added D6: STATUS, Custom:LED_THT_L72CB_Kingbright, B.Cu at (118.1, 226.0)
- added E1: ~, Custom:Hammond_Enclosure_RM2095L, F.Cu at (196.5, 139.8)
- added J11: SPARE, Connector_PinHeader_2.54mm:PinHeader_1x05_P2.54mm_Vertical, F.Cu at (287.0, 61.0)
- added J15: SERIAL, Connector_PinHeader_2.54mm:PinHeader_1x06_P2.54mm_Vertical, F.Cu at (135.9, 62.2)
- added J19: SPARE, Connector_PinHeader_2.54mm:PinHeader_1x05_P2.54mm_Vertical, F.Cu at (287.0, 63.5)
- added J20: RVLINK, Connector_PinHeader_2.54mm:PinHeader_1x02_P2.54mm_Vertical, F.Cu at (191.8, 73.7)
- added J23: ANALOG, Connector_PinHeader_2.54mm:PinHeader_1x04_P2.54mm_Vertical, F.Cu at (255.5, 108.2)
- added J24: ANALOG, Connector_PinHeader_2.54mm:PinHeader_1x04_P2.54mm_Vertical, F.Cu at (255.5, 131.1)
- added J25: EXP, Connector_PinHeader_2.54mm:PinHeader_1x16_P2.54mm_Vertical, F.Cu at (179.7, 126.4)
- added J4: SERIAL, TerminalBlock_Phoenix:TerminalBlock_Phoenix_PT-1,5-6-3.5-H_1x06_P3.50mm_Horizontal, F.Cu at (130.5, 44.5)
- added J7: SPARE, TerminalBlock_Phoenix:TerminalBlock_Phoenix_PT-1,5-5-3.5-H_1x05_P3.50mm_Horizontal, F.Cu at (288.6, 44.5)
- added J9: PGND, Connector_PinHeader_2.54mm:PinHeader_2x02_P2.54mm_Vertical, F.Cu at (295.7, 92.5)
- added L1: 100uH, Inductor_THT:L_Axial_L9.5mm_D4.0mm_P5.08mm_Vertical_Fastron_SMCC, F.Cu at (281.9, 86.9)
- added L2: 100uH, Inductor_THT:L_Axial_L9.5mm_D4.0mm_P5.08mm_Vertical_Fastron_SMCC, F.Cu at (264.2, 86.9)
- added L3: 100uH, Inductor_THT:L_Axial_L9.5mm_D4.0mm_P5.08mm_Vertical_Fastron_SMCC, F.Cu at (281.9, 100.3)
- added L4: 100uH, Inductor_THT:L_Axial_L9.5mm_D4.0mm_P5.08mm_Vertical_Fastron_SMCC, F.Cu at (264.2, 100.3)
- added PR1: ~, Custom:Prototype Area 5x13 with 4 rails (5x17) 2.54mm Grid, F.Cu at (167.6, 161.9)
- added PR2: ~, Custom:Prototype Area 5x13 with 4 rails (5x17) 2.54mm Grid, F.Cu at (154.9, 161.9)
- added PR3: ~, Custom:Prototype Area 5x13 with 4 rails (5x17) 2.54mm Grid, F.Cu at (142.2, 161.9)
- added PR4: ~, Custom:Prototype Area 5x13 with 4 rails (5x17) 2.54mm Grid, F.Cu at (116.8, 161.9)
- added PR5: ~, Custom:Prototype Area 5x13 with 4 rails (5x17) 2.54mm Grid, F.Cu at (129.5, 161.9)
- added Q1: BC547, Package_TO_SOT_THT:TO-92L_Wide, F.Cu at (278.9, 123.2)
- added R1: 1K, Resistor_THT:R_Axial_DIN0207_L6.3mm_D2.5mm_P10.16mm_Horizontal, F.Cu at (185.4, 95.2)
- added R14: 1K, Resistor_THT:R_Axial_DIN0207_L6.3mm_D2.5mm_P10.16mm_Horizontal, F.Cu at (261.6, 129.5)
- added R15: 1K, Resistor_THT:R_Axial_DIN0207_L6.3mm_D2.5mm_P10.16mm_Horizontal, F.Cu at (261.6, 125.7)
- added R17: 1K, Resistor_THT:R_Axial_DIN0207_L6.3mm_D2.5mm_P10.16mm_Horizontal, F.Cu at (96.5, 187.3)
- added R18: 390R, Resistor_THT:R_Axial_DIN0207_L6.3mm_D2.5mm_P10.16mm_Horizontal, F.Cu at (108.0, 187.3)
- added R19: 1K, Resistor_THT:R_Axial_DIN0207_L6.3mm_D2.5mm_P10.16mm_Horizontal, F.Cu at (104.1, 187.3)
- added R2: 1K, Resistor_THT:R_Axial_DIN0207_L6.3mm_D2.5mm_P10.16mm_Horizontal, F.Cu at (181.6, 95.2)
- added R20: 1K, Resistor_THT:R_Axial_DIN0207_L6.3mm_D2.5mm_P10.16mm_Horizontal, F.Cu at (100.3, 187.3)
- added R3: 1K, Resistor_THT:R_Axial_DIN0207_L6.3mm_D2.5mm_P10.16mm_Horizontal, F.Cu at (193.0, 121.9)
- added R4: 1K, Resistor_THT:R_Axial_DIN0207_L6.3mm_D2.5mm_P10.16mm_Horizontal, F.Cu at (189.2, 121.9)
- added R53: 1K, Resistor_THT:R_Axial_DIN0207_L6.3mm_D2.5mm_P10.16mm_Horizontal, F.Cu at (149.9, 214.6)
- added R54: 1K, Resistor_THT:R_Axial_DIN0207_L6.3mm_D2.5mm_P10.16mm_Horizontal, F.Cu at (160.0, 214.6)
- added R55: 1K, Resistor_THT:R_Axial_DIN0207_L6.3mm_D2.5mm_P10.16mm_Horizontal, F.Cu at (170.2, 214.6)
- added R56: 1K, Resistor_THT:R_Axial_DIN0207_L6.3mm_D2.5mm_P10.16mm_Horizontal, F.Cu at (180.3, 214.6)
- added R57: 1K, Resistor_THT:R_Axial_DIN0207_L6.3mm_D2.5mm_P10.16mm_Horizontal, F.Cu at (190.5, 214.6)
- added R58: 1K, Resistor_THT:R_Axial_DIN0207_L6.3mm_D2.5mm_P10.16mm_Horizontal, F.Cu at (200.7, 214.6)
- added R59: 1K, Resistor_THT:R_Axial_DIN0207_L6.3mm_D2.5mm_P10.16mm_Horizontal, F.Cu at (219.7, 214.6)
- added R6: 1K, Resistor_THT:R_Axial_DIN0207_L6.3mm_D2.5mm_P10.16mm_Horizontal, F.Cu at (189.2, 95.2)
- added R60: 1K, Resistor_THT:R_Axial_DIN0207_L6.3mm_D2.5mm_P10.16mm_Horizontal, F.Cu at (229.9, 214.6)
- added R61: 1K, Resistor_THT:R_Axial_DIN0207_L6.3mm_D2.5mm_P10.16mm_Horizontal, F.Cu at (240.0, 214.6)
- added R62: 1K, Resistor_THT:R_Axial_DIN0207_L6.3mm_D2.5mm_P10.16mm_Horizontal, F.Cu at (250.2, 214.6)
- added R63: 1K, Resistor_THT:R_Axial_DIN0207_L6.3mm_D2.5mm_P10.16mm_Horizontal, F.Cu at (260.4, 214.6)
- added R64: 1K, Resistor_THT:R_Axial_DIN0207_L6.3mm_D2.5mm_P10.16mm_Horizontal, F.Cu at (270.5, 214.6)
- added R8: 1K, Resistor_THT:R_Axial_DIN0207_L6.3mm_D2.5mm_P10.16mm_Horizontal, F.Cu at (287.0, 91.4)
- added REF**: Pad_D1.5mm_Drill1.0mm, RF_Custom:Pad_D1.5mm_Drill1.0mm, F.Cu at (137.2, 215.9)
- added REF**: Pad_D1.5mm_Drill1.0mm, RF_Custom:Pad_D1.5mm_Drill1.0mm, F.Cu at (109.2, 116.8)
- added REF**: Pad_D1.5mm_Drill1.0mm, RF_Custom:Pad_D1.5mm_Drill1.0mm, F.Cu at (124.5, 228.6)
- added REF**: Pad_D1.5mm_Drill1.0mm, RF_Custom:Pad_D1.5mm_Drill1.0mm, F.Cu at (149.9, 114.3)
- added REF**: Pad_D1.5mm_Drill1.0mm, RF_Custom:Pad_D1.5mm_Drill1.0mm, F.Cu at (124.5, 185.4)
- added REF**: Pad_D1.5mm_Drill1.0mm, RF_Custom:Pad_D1.5mm_Drill1.0mm, F.Cu at (137.2, 203.2)
- added REF**: Pad_D1.5mm_Drill1.0mm, RF_Custom:Pad_D1.5mm_Drill1.0mm, F.Cu at (121.8, 177.6)
- added REF**: Pad_D1.5mm_Drill1.0mm, RF_Custom:Pad_D1.5mm_Drill1.0mm, F.Cu at (149.9, 106.7)
- added REF**: Pad_D1.5mm_Drill1.0mm, RF_Custom:Pad_D1.5mm_Drill1.0mm, F.Cu at (139.7, 198.1)
- added REF**: Pad_D1.5mm_Drill1.0mm, RF_Custom:Pad_D1.5mm_Drill1.0mm, F.Cu at (124.5, 231.1)
- added REF**: Pad_D1.5mm_Drill1.0mm, RF_Custom:Pad_D1.5mm_Drill1.0mm, F.Cu at (134.6, 190.5)
- added REF**: Pad_D1.5mm_Drill1.0mm, RF_Custom:Pad_D1.5mm_Drill1.0mm, F.Cu at (121.9, 236.2)
- added REF**: Pad_D1.5mm_Drill1.0mm, RF_Custom:Pad_D1.5mm_Drill1.0mm, F.Cu at (121.9, 185.4)
- added REF**: Pad_D1.5mm_Drill1.0mm, RF_Custom:Pad_D1.5mm_Drill1.0mm, F.Cu at (134.6, 205.7)
- added REF**: Pad_D1.5mm_Drill1.0mm, RF_Custom:Pad_D1.5mm_Drill1.0mm, F.Cu at (139.7, 208.3)
- added REF**: Pad_D1.5mm_Drill1.0mm, RF_Custom:Pad_D1.5mm_Drill1.0mm, F.Cu at (124.4, 172.7)
- added REF**: Pad_D1.5mm_Drill1.0mm, RF_Custom:Pad_D1.5mm_Drill1.0mm, F.Cu at (137.2, 233.7)
- added REF**: Pad_D1.5mm_Drill1.0mm, RF_Custom:Pad_D1.5mm_Drill1.0mm, F.Cu at (129.4, 177.6)
- added REF**: Pad_D1.5mm_Drill1.0mm, RF_Custom:Pad_D1.5mm_Drill1.0mm, F.Cu at (129.5, 111.8)
- added REF**: Pad_D1.5mm_Drill1.0mm, RF_Custom:Pad_D1.5mm_Drill1.0mm, F.Cu at (121.9, 218.4)
- added REF**: Pad_D1.5mm_Drill1.0mm, RF_Custom:Pad_D1.5mm_Drill1.0mm, F.Cu at (121.9, 233.7)
- added REF**: Pad_D1.5mm_Drill1.0mm, RF_Custom:Pad_D1.5mm_Drill1.0mm, F.Cu at (124.4, 177.6)
- added REF**: Pad_D1.5mm_Drill1.0mm, RF_Custom:Pad_D1.5mm_Drill1.0mm, F.Cu at (124.5, 182.9)
- added REF**: Pad_D1.5mm_Drill1.0mm, RF_Custom:Pad_D1.5mm_Drill1.0mm, F.Cu at (139.7, 236.2)
- added REF**: Pad_D1.5mm_Drill1.0mm, RF_Custom:Pad_D1.5mm_Drill1.0mm, F.Cu at (137.2, 223.5)
- added REF**: Pad_D1.5mm_Drill1.0mm, RF_Custom:Pad_D1.5mm_Drill1.0mm, F.Cu at (132.1, 208.3)
- added REF**: Pad_D1.5mm_Drill1.0mm, RF_Custom:Pad_D1.5mm_Drill1.0mm, F.Cu at (124.5, 208.3)
- added REF**: Pad_D1.5mm_Drill1.0mm, RF_Custom:Pad_D1.5mm_Drill1.0mm, F.Cu at (132.1, 182.9)
- added REF**: Pad_D1.5mm_Drill1.0mm, RF_Custom:Pad_D1.5mm_Drill1.0mm, F.Cu at (114.3, 106.7)
- added REF**: Pad_D1.5mm_Drill1.0mm, RF_Custom:Pad_D1.5mm_Drill1.0mm, F.Cu at (121.9, 111.8)
- added REF**: Pad_D1.5mm_Drill1.0mm, RF_Custom:Pad_D1.5mm_Drill1.0mm, F.Cu at (127.0, 180.3)
- added REF**: Pad_D1.5mm_Drill1.0mm, RF_Custom:Pad_D1.5mm_Drill1.0mm, F.Cu at (129.5, 182.9)
- added REF**: Pad_D1.5mm_Drill1.0mm, RF_Custom:Pad_D1.5mm_Drill1.0mm, F.Cu at (139.7, 203.2)
- added REF**: Pad_D1.5mm_Drill1.0mm, RF_Custom:Pad_D1.5mm_Drill1.0mm, F.Cu at (129.5, 190.5)
- added REF**: Pad_D1.5mm_Drill1.0mm, RF_Custom:Pad_D1.5mm_Drill1.0mm, F.Cu at (139.7, 215.9)
- added REF**: Pad_D1.5mm_Drill1.0mm, RF_Custom:Pad_D1.5mm_Drill1.0mm, F.Cu at (139.7, 205.7)
- added REF**: Pad_D1.5mm_Drill1.0mm, RF_Custom:Pad_D1.5mm_Drill1.0mm, F.Cu at (124.5, 190.5)
- added REF**: Pad_D1.5mm_Drill1.0mm, RF_Custom:Pad_D1.5mm_Drill1.0mm, F.Cu at (134.6, 182.9)
- added REF**: Pad_D1.5mm_Drill1.0mm, RF_Custom:Pad_D1.5mm_Drill1.0mm, F.Cu at (126.9, 175.3)
- added REF**: Pad_D1.5mm_Drill1.0mm, RF_Custom:Pad_D1.5mm_Drill1.0mm, F.Cu at (132.1, 213.4)
- added REF**: Pad_D1.5mm_Drill1.0mm, RF_Custom:Pad_D1.5mm_Drill1.0mm, F.Cu at (121.9, 221.0)
- added REF**: Pad_D1.5mm_Drill1.0mm, RF_Custom:Pad_D1.5mm_Drill1.0mm, F.Cu at (127.0, 111.8)
- added REF**: Pad_D1.5mm_Drill1.0mm, RF_Custom:Pad_D1.5mm_Drill1.0mm, F.Cu at (127.0, 218.4)
- added REF**: Pad_D1.5mm_Drill1.0mm, RF_Custom:Pad_D1.5mm_Drill1.0mm, F.Cu at (137.2, 226.1)
- added REF**: Pad_D1.5mm_Drill1.0mm, RF_Custom:Pad_D1.5mm_Drill1.0mm, F.Cu at (147.3, 116.8)
- added REF**: Pad_D1.5mm_Drill1.0mm, RF_Custom:Pad_D1.5mm_Drill1.0mm, F.Cu at (127.0, 198.1)
- added REF**: Pad_D1.5mm_Drill1.0mm, RF_Custom:Pad_D1.5mm_Drill1.0mm, F.Cu at (132.1, 236.2)
- added REF**: Pad_D1.5mm_Drill1.0mm, RF_Custom:Pad_D1.5mm_Drill1.0mm, F.Cu at (152.4, 116.8)
- added REF**: Pad_D1.5mm_Drill1.0mm, RF_Custom:Pad_D1.5mm_Drill1.0mm, F.Cu at (109.2, 109.2)
- added REF**: Pad_D1.5mm_Drill1.0mm, RF_Custom:Pad_D1.5mm_Drill1.0mm, F.Cu at (134.6, 228.6)
- added REF**: Pad_D1.5mm_Drill1.0mm, RF_Custom:Pad_D1.5mm_Drill1.0mm, F.Cu at (129.5, 116.8)
- added REF**: Pad_D1.5mm_Drill1.0mm, RF_Custom:Pad_D1.5mm_Drill1.0mm, F.Cu at (129.5, 210.8)
- added REF**: Pad_D1.5mm_Drill1.0mm, RF_Custom:Pad_D1.5mm_Drill1.0mm, F.Cu at (114.3, 111.8)
- added REF**: Pad_D1.5mm_Drill1.0mm, RF_Custom:Pad_D1.5mm_Drill1.0mm, F.Cu at (132.1, 111.8)
- added REF**: Pad_D1.5mm_Drill1.0mm, RF_Custom:Pad_D1.5mm_Drill1.0mm, F.Cu at (127.0, 226.1)
- added REF**: Pad_D1.5mm_Drill1.0mm, RF_Custom:Pad_D1.5mm_Drill1.0mm, F.Cu at (127.0, 106.7)
- added REF**: Pad_D1.5mm_Drill1.0mm, RF_Custom:Pad_D1.5mm_Drill1.0mm, F.Cu at (142.2, 111.8)
- added REF**: Pad_D1.5mm_Drill1.0mm, RF_Custom:Pad_D1.5mm_Drill1.0mm, F.Cu at (139.7, 190.5)
- added REF**: Pad_D1.5mm_Drill1.0mm, RF_Custom:Pad_D1.5mm_Drill1.0mm, F.Cu at (132.1, 114.3)
- added REF**: Pad_D1.5mm_Drill1.0mm, RF_Custom:Pad_D1.5mm_Drill1.0mm, F.Cu at (129.5, 226.1)
- added REF**: Pad_D1.5mm_Drill1.0mm, RF_Custom:Pad_D1.5mm_Drill1.0mm, F.Cu at (132.1, 228.6)
- added REF**: Pad_D1.5mm_Drill1.0mm, RF_Custom:Pad_D1.5mm_Drill1.0mm, F.Cu at (129.5, 203.2)
- added REF**: Pad_D1.5mm_Drill1.0mm, RF_Custom:Pad_D1.5mm_Drill1.0mm, F.Cu at (132.1, 180.3)
- added REF**: Pad_D1.5mm_Drill1.0mm, RF_Custom:Pad_D1.5mm_Drill1.0mm, F.Cu at (134.6, 111.8)
- added REF**: Pad_D1.5mm_Drill1.0mm, RF_Custom:Pad_D1.5mm_Drill1.0mm, F.Cu at (116.8, 106.7)
- added REF**: Pad_D1.5mm_Drill1.0mm, RF_Custom:Pad_D1.5mm_Drill1.0mm, F.Cu at (137.2, 185.4)
- added REF**: Pad_D1.5mm_Drill1.0mm, RF_Custom:Pad_D1.5mm_Drill1.0mm, F.Cu at (152.4, 114.3)
- added REF**: Pad_D1.5mm_Drill1.0mm, RF_Custom:Pad_D1.5mm_Drill1.0mm, F.Cu at (132.1, 215.9)
- added REF**: Pad_D1.5mm_Drill1.0mm, RF_Custom:Pad_D1.5mm_Drill1.0mm, F.Cu at (137.2, 221.0)
- added REF**: Pad_D1.5mm_Drill1.0mm, RF_Custom:Pad_D1.5mm_Drill1.0mm, F.Cu at (129.5, 195.6)
- added REF**: Pad_D1.5mm_Drill1.0mm, RF_Custom:Pad_D1.5mm_Drill1.0mm, F.Cu at (121.9, 182.9)
- added REF**: Pad_D1.5mm_Drill1.0mm, RF_Custom:Pad_D1.5mm_Drill1.0mm, F.Cu at (149.9, 109.2)
- added REF**: Pad_D1.5mm_Drill1.0mm, RF_Custom:Pad_D1.5mm_Drill1.0mm, F.Cu at (119.4, 111.8)
- added REF**: Pad_D1.5mm_Drill1.0mm, RF_Custom:Pad_D1.5mm_Drill1.0mm, F.Cu at (121.9, 190.5)
- added REF**: Pad_D1.5mm_Drill1.0mm, RF_Custom:Pad_D1.5mm_Drill1.0mm, F.Cu at (139.7, 210.8)
- added REF**: Pad_D1.5mm_Drill1.0mm, RF_Custom:Pad_D1.5mm_Drill1.0mm, F.Cu at (132.1, 223.5)
- added REF**: Pad_D1.5mm_Drill1.0mm, RF_Custom:Pad_D1.5mm_Drill1.0mm, F.Cu at (137.2, 193.0)
- added REF**: Pad_D1.5mm_Drill1.0mm, RF_Custom:Pad_D1.5mm_Drill1.0mm, F.Cu at (124.5, 218.4)
- added REF**: Pad_D1.5mm_Drill1.0mm, RF_Custom:Pad_D1.5mm_Drill1.0mm, F.Cu at (139.7, 106.7)
- added REF**: Pad_D1.5mm_Drill1.0mm, RF_Custom:Pad_D1.5mm_Drill1.0mm, F.Cu at (129.5, 185.4)
- added REF**: Pad_D1.5mm_Drill1.0mm, RF_Custom:Pad_D1.5mm_Drill1.0mm, F.Cu at (111.8, 109.2)
- added REF**: Pad_D1.5mm_Drill1.0mm, RF_Custom:Pad_D1.5mm_Drill1.0mm, F.Cu at (119.4, 114.3)
- added REF**: Pad_D1.5mm_Drill1.0mm, RF_Custom:Pad_D1.5mm_Drill1.0mm, F.Cu at (124.4, 175.3)
- added REF**: Pad_D1.5mm_Drill1.0mm, RF_Custom:Pad_D1.5mm_Drill1.0mm, F.Cu at (132.1, 233.7)
- added REF**: Pad_D1.5mm_Drill1.0mm, RF_Custom:Pad_D1.5mm_Drill1.0mm, F.Cu at (114.3, 114.3)
- added REF**: Pad_D1.5mm_Drill1.0mm, RF_Custom:Pad_D1.5mm_Drill1.0mm, F.Cu at (127.0, 231.1)
- added REF**: Pad_D1.5mm_Drill1.0mm, RF_Custom:Pad_D1.5mm_Drill1.0mm, F.Cu at (144.8, 111.8)
- added REF**: Pad_D1.5mm_Drill1.0mm, RF_Custom:Pad_D1.5mm_Drill1.0mm, F.Cu at (134.6, 198.1)
- added REF**: Pad_D1.5mm_Drill1.0mm, RF_Custom:Pad_D1.5mm_Drill1.0mm, F.Cu at (116.8, 111.8)
- added REF**: Pad_D1.5mm_Drill1.0mm, RF_Custom:Pad_D1.5mm_Drill1.0mm, F.Cu at (124.5, 221.0)
- added REF**: Pad_D1.5mm_Drill1.0mm, RF_Custom:Pad_D1.5mm_Drill1.0mm, F.Cu at (116.8, 109.2)
- added REF**: Pad_D1.5mm_Drill1.0mm, RF_Custom:Pad_D1.5mm_Drill1.0mm, F.Cu at (137.2, 114.3)
- added REF**: Pad_D1.5mm_Drill1.0mm, RF_Custom:Pad_D1.5mm_Drill1.0mm, F.Cu at (124.5, 213.4)
- added REF**: Pad_D1.5mm_Drill1.0mm, RF_Custom:Pad_D1.5mm_Drill1.0mm, F.Cu at (132.1, 231.1)
- added REF**: Pad_D1.5mm_Drill1.0mm, RF_Custom:Pad_D1.5mm_Drill1.0mm, F.Cu at (116.8, 114.3)
- added REF**: Pad_D1.5mm_Drill1.0mm, RF_Custom:Pad_D1.5mm_Drill1.0mm, F.Cu at (152.4, 106.7)
- added REF**: Pad_D1.5mm_Drill1.0mm, RF_Custom:Pad_D1.5mm_Drill1.0mm, F.Cu at (124.5, 205.7)
- added REF**: Pad_D1.5mm_Drill1.0mm, RF_Custom:Pad_D1.5mm_Drill1.0mm, F.Cu at (139.7, 228.6)
- added REF**: Pad_D1.5mm_Drill1.0mm, RF_Custom:Pad_D1.5mm_Drill1.0mm, F.Cu at (129.5, 215.9)
- added REF**: Pad_D1.5mm_Drill1.0mm, RF_Custom:Pad_D1.5mm_Drill1.0mm, F.Cu at (137.2, 231.1)
- added REF**: Pad_D1.5mm_Drill1.0mm, RF_Custom:Pad_D1.5mm_Drill1.0mm, F.Cu at (127.0, 223.5)
- added REF**: Pad_D1.5mm_Drill1.0mm, RF_Custom:Pad_D1.5mm_Drill1.0mm, F.Cu at (132.1, 106.7)
- added REF**: Pad_D1.5mm_Drill1.0mm, RF_Custom:Pad_D1.5mm_Drill1.0mm, F.Cu at (129.5, 200.7)
- added REF**: Pad_D1.5mm_Drill1.0mm, RF_Custom:Pad_D1.5mm_Drill1.0mm, F.Cu at (139.7, 114.3)
- added REF**: Pad_D1.5mm_Drill1.0mm, RF_Custom:Pad_D1.5mm_Drill1.0mm, F.Cu at (132.1, 116.8)
- added REF**: Pad_D1.5mm_Drill1.0mm, RF_Custom:Pad_D1.5mm_Drill1.0mm, F.Cu at (124.5, 233.7)
- added REF**: Pad_D1.5mm_Drill1.0mm, RF_Custom:Pad_D1.5mm_Drill1.0mm, F.Cu at (137.1, 170.2)
- added REF**: Pad_D1.5mm_Drill1.0mm, RF_Custom:Pad_D1.5mm_Drill1.0mm, F.Cu at (121.9, 226.1)
- added REF**: Pad_D1.5mm_Drill1.0mm, RF_Custom:Pad_D1.5mm_Drill1.0mm, F.Cu at (134.6, 106.7)
- added REF**: Pad_D1.5mm_Drill1.0mm, RF_Custom:Pad_D1.5mm_Drill1.0mm, F.Cu at (129.5, 205.7)
- added REF**: Pad_D1.5mm_Drill1.0mm, RF_Custom:Pad_D1.5mm_Drill1.0mm, F.Cu at (147.3, 109.2)
- added REF**: Pad_D1.5mm_Drill1.0mm, RF_Custom:Pad_D1.5mm_Drill1.0mm, F.Cu at (139.7, 185.4)
- added REF**: Pad_D1.5mm_Drill1.0mm, RF_Custom:Pad_D1.5mm_Drill1.0mm, F.Cu at (134.6, 226.1)
- added REF**: Pad_D1.5mm_Drill1.0mm, RF_Custom:Pad_D1.5mm_Drill1.0mm, F.Cu at (137.2, 198.1)
- added REF**: Pad_D1.5mm_Drill1.0mm, RF_Custom:Pad_D1.5mm_Drill1.0mm, F.Cu at (132.1, 205.7)
- added REF**: Pad_D1.5mm_Drill1.0mm, RF_Custom:Pad_D1.5mm_Drill1.0mm, F.Cu at (129.5, 236.2)
- added REF**: Pad_D1.5mm_Drill1.0mm, RF_Custom:Pad_D1.5mm_Drill1.0mm, F.Cu at (129.4, 170.2)
- added REF**: Pad_D1.5mm_Drill1.0mm, RF_Custom:Pad_D1.5mm_Drill1.0mm, F.Cu at (139.7, 200.7)
- added REF**: Pad_D1.5mm_Drill1.0mm, RF_Custom:Pad_D1.5mm_Drill1.0mm, F.Cu at (144.8, 233.7)
- added REF**: Pad_D1.5mm_Drill1.0mm, RF_Custom:Pad_D1.5mm_Drill1.0mm, F.Cu at (142.2, 236.2)
- added REF**: Pad_D1.5mm_Drill1.0mm, RF_Custom:Pad_D1.5mm_Drill1.0mm, F.Cu at (121.9, 231.1)
- added REF**: Pad_D1.5mm_Drill1.0mm, RF_Custom:Pad_D1.5mm_Drill1.0mm, F.Cu at (124.5, 180.3)
- added REF**: Pad_D1.5mm_Drill1.0mm, RF_Custom:Pad_D1.5mm_Drill1.0mm, F.Cu at (129.5, 228.6)
- added REF**: Pad_D1.5mm_Drill1.0mm, RF_Custom:Pad_D1.5mm_Drill1.0mm, F.Cu at (137.2, 111.8)
- added REF**: Pad_D1.5mm_Drill1.0mm, RF_Custom:Pad_D1.5mm_Drill1.0mm, F.Cu at (132.0, 172.7)
- added REF**: Pad_D1.5mm_Drill1.0mm, RF_Custom:Pad_D1.5mm_Drill1.0mm, F.Cu at (137.2, 200.7)
- added REF**: Pad_D1.5mm_Drill1.0mm, RF_Custom:Pad_D1.5mm_Drill1.0mm, F.Cu at (137.2, 116.8)
- added REF**: Pad_D1.5mm_Drill1.0mm, RF_Custom:Pad_D1.5mm_Drill1.0mm, F.Cu at (134.5, 175.3)
- added REF**: Pad_D1.5mm_Drill1.0mm, RF_Custom:Pad_D1.5mm_Drill1.0mm, F.Cu at (144.8, 116.8)
- added REF**: Pad_D1.5mm_Drill1.0mm, RF_Custom:Pad_D1.5mm_Drill1.0mm, F.Cu at (139.7, 218.4)
- added REF**: Pad_D1.5mm_Drill1.0mm, RF_Custom:Pad_D1.5mm_Drill1.0mm, F.Cu at (121.9, 223.5)
- added REF**: Pad_D1.5mm_Drill1.0mm, RF_Custom:Pad_D1.5mm_Drill1.0mm, F.Cu at (121.9, 198.1)
- added REF**: Pad_D1.5mm_Drill1.0mm, RF_Custom:Pad_D1.5mm_Drill1.0mm, F.Cu at (132.1, 226.1)
- added REF**: Pad_D1.5mm_Drill1.0mm, RF_Custom:Pad_D1.5mm_Drill1.0mm, F.Cu at (152.4, 111.8)
- added REF**: Pad_D1.5mm_Drill1.0mm, RF_Custom:Pad_D1.5mm_Drill1.0mm, F.Cu at (129.5, 198.1)
- added REF**: Pad_D1.5mm_Drill1.0mm, RF_Custom:Pad_D1.5mm_Drill1.0mm, F.Cu at (132.1, 221.0)
- added REF**: Pad_D1.5mm_Drill1.0mm, RF_Custom:Pad_D1.5mm_Drill1.0mm, F.Cu at (147.3, 106.7)
- added REF**: Pad_D1.5mm_Drill1.0mm, RF_Custom:Pad_D1.5mm_Drill1.0mm, F.Cu at (132.0, 177.6)
- added REF**: Pad_D1.5mm_Drill1.0mm, RF_Custom:Pad_D1.5mm_Drill1.0mm, F.Cu at (121.9, 228.6)
- added REF**: Pad_D1.5mm_Drill1.0mm, RF_Custom:Pad_D1.5mm_Drill1.0mm, F.Cu at (129.5, 218.4)
- added REF**: Pad_D1.5mm_Drill1.0mm, RF_Custom:Pad_D1.5mm_Drill1.0mm, F.Cu at (139.7, 180.3)
- added REF**: Pad_D1.5mm_Drill1.0mm, RF_Custom:Pad_D1.5mm_Drill1.0mm, F.Cu at (121.9, 208.3)
- added REF**: Pad_D1.5mm_Drill1.0mm, RF_Custom:Pad_D1.5mm_Drill1.0mm, F.Cu at (142.2, 228.6)
- added REF**: Pad_D1.5mm_Drill1.0mm, RF_Custom:Pad_D1.5mm_Drill1.0mm, F.Cu at (121.9, 195.6)
- added REF**: Pad_D1.5mm_Drill1.0mm, RF_Custom:Pad_D1.5mm_Drill1.0mm, F.Cu at (134.6, 193.0)
- added REF**: Pad_D1.5mm_Drill1.0mm, RF_Custom:Pad_D1.5mm_Drill1.0mm, F.Cu at (109.2, 111.8)
- added REF**: Pad_D1.5mm_Drill1.0mm, RF_Custom:Pad_D1.5mm_Drill1.0mm, F.Cu at (124.5, 188.0)
- added REF**: Pad_D1.5mm_Drill1.0mm, RF_Custom:Pad_D1.5mm_Drill1.0mm, F.Cu at (129.5, 114.3)
- added REF**: Pad_D1.5mm_Drill1.0mm, RF_Custom:Pad_D1.5mm_Drill1.0mm, F.Cu at (152.4, 109.2)
- added REF**: Pad_D1.5mm_Drill1.0mm, RF_Custom:Pad_D1.5mm_Drill1.0mm, F.Cu at (139.7, 226.1)
- added REF**: Pad_D1.5mm_Drill1.0mm, RF_Custom:Pad_D1.5mm_Drill1.0mm, F.Cu at (137.2, 188.0)
- added REF**: Pad_D1.5mm_Drill1.0mm, RF_Custom:Pad_D1.5mm_Drill1.0mm, F.Cu at (137.2, 228.6)
- added REF**: Pad_D1.5mm_Drill1.0mm, RF_Custom:Pad_D1.5mm_Drill1.0mm, F.Cu at (144.8, 231.1)
- added REF**: Pad_D1.5mm_Drill1.0mm, RF_Custom:Pad_D1.5mm_Drill1.0mm, F.Cu at (137.2, 218.4)
- added REF**: Pad_D1.5mm_Drill1.0mm, RF_Custom:Pad_D1.5mm_Drill1.0mm, F.Cu at (129.5, 223.5)
- added REF**: Pad_D1.5mm_Drill1.0mm, RF_Custom:Pad_D1.5mm_Drill1.0mm, F.Cu at (124.5, 200.7)
- added REF**: Pad_D1.5mm_Drill1.0mm, RF_Custom:Pad_D1.5mm_Drill1.0mm, F.Cu at (142.2, 106.7)
- added REF**: Pad_D1.5mm_Drill1.0mm, RF_Custom:Pad_D1.5mm_Drill1.0mm, F.Cu at (121.8, 172.7)
- added REF**: Pad_D1.5mm_Drill1.0mm, RF_Custom:Pad_D1.5mm_Drill1.0mm, F.Cu at (124.5, 114.3)
- added REF**: Pad_D1.5mm_Drill1.0mm, RF_Custom:Pad_D1.5mm_Drill1.0mm, F.Cu at (144.8, 236.2)
- added REF**: Pad_D1.5mm_Drill1.0mm, RF_Custom:Pad_D1.5mm_Drill1.0mm, F.Cu at (111.8, 111.8)
- added REF**: Pad_D1.5mm_Drill1.0mm, RF_Custom:Pad_D1.5mm_Drill1.0mm, F.Cu at (134.6, 223.5)
- added REF**: Pad_D1.5mm_Drill1.0mm, RF_Custom:Pad_D1.5mm_Drill1.0mm, F.Cu at (134.5, 177.6)
- added REF**: Pad_D1.5mm_Drill1.0mm, RF_Custom:Pad_D1.5mm_Drill1.0mm, F.Cu at (121.9, 210.8)
- added REF**: Pad_D1.5mm_Drill1.0mm, RF_Custom:Pad_D1.5mm_Drill1.0mm, F.Cu at (142.2, 233.7)
- added REF**: Pad_D1.5mm_Drill1.0mm, RF_Custom:Pad_D1.5mm_Drill1.0mm, F.Cu at (142.2, 114.3)
- added REF**: Pad_D1.5mm_Drill1.0mm, RF_Custom:Pad_D1.5mm_Drill1.0mm, F.Cu at (127.0, 221.0)
- added REF**: Pad_D1.5mm_Drill1.0mm, RF_Custom:Pad_D1.5mm_Drill1.0mm, F.Cu at (134.6, 188.0)
- added REF**: Pad_D1.5mm_Drill1.0mm, RF_Custom:Pad_D1.5mm_Drill1.0mm, F.Cu at (121.9, 203.2)
- added REF**: Pad_D1.5mm_Drill1.0mm, RF_Custom:Pad_D1.5mm_Drill1.0mm, F.Cu at (132.1, 190.5)
- added REF**: Pad_D1.5mm_Drill1.0mm, RF_Custom:Pad_D1.5mm_Drill1.0mm, F.Cu at (121.9, 215.9)
- added REF**: Pad_D1.5mm_Drill1.0mm, RF_Custom:Pad_D1.5mm_Drill1.0mm, F.Cu at (137.2, 210.8)
- added REF**: Pad_D1.5mm_Drill1.0mm, RF_Custom:Pad_D1.5mm_Drill1.0mm, F.Cu at (126.9, 172.7)
- added REF**: Pad_D1.5mm_Drill1.0mm, RF_Custom:Pad_D1.5mm_Drill1.0mm, F.Cu at (132.1, 188.0)
- added REF**: Pad_D1.5mm_Drill1.0mm, RF_Custom:Pad_D1.5mm_Drill1.0mm, F.Cu at (126.9, 177.6)
- added REF**: Pad_D1.5mm_Drill1.0mm, RF_Custom:Pad_D1.5mm_Drill1.0mm, F.Cu at (137.1, 175.3)
- added REF**: Pad_D1.5mm_Drill1.0mm, RF_Custom:Pad_D1.5mm_Drill1.0mm, F.Cu at (124.5, 226.1)
- added REF**: Pad_D1.5mm_Drill1.0mm, RF_Custom:Pad_D1.5mm_Drill1.0mm, F.Cu at (149.9, 116.8)
- added REF**: Pad_D1.5mm_Drill1.0mm, RF_Custom:Pad_D1.5mm_Drill1.0mm, F.Cu at (119.4, 116.8)
- added REF**: Pad_D1.5mm_Drill1.0mm, RF_Custom:Pad_D1.5mm_Drill1.0mm, F.Cu at (144.8, 109.2)
- added REF**: Pad_D1.5mm_Drill1.0mm, RF_Custom:Pad_D1.5mm_Drill1.0mm, F.Cu at (132.1, 109.2)
- added REF**: Pad_D1.5mm_Drill1.0mm, RF_Custom:Pad_D1.5mm_Drill1.0mm, F.Cu at (124.4, 170.2)
- added REF**: Pad_D1.5mm_Drill1.0mm, RF_Custom:Pad_D1.5mm_Drill1.0mm, F.Cu at (127.0, 114.3)
- added REF**: Pad_D1.5mm_Drill1.0mm, RF_Custom:Pad_D1.5mm_Drill1.0mm, F.Cu at (132.1, 203.2)
- added REF**: Pad_D1.5mm_Drill1.0mm, RF_Custom:Pad_D1.5mm_Drill1.0mm, F.Cu at (121.9, 200.7)
- added REF**: Pad_D1.5mm_Drill1.0mm, RF_Custom:Pad_D1.5mm_Drill1.0mm, F.Cu at (144.8, 114.3)
- added REF**: Pad_D1.5mm_Drill1.0mm, RF_Custom:Pad_D1.5mm_Drill1.0mm, F.Cu at (139.7, 116.8)
- added REF**: Pad_D1.5mm_Drill1.0mm, RF_Custom:Pad_D1.5mm_Drill1.0mm, F.Cu at (139.6, 175.3)
- added REF**: Pad_D1.5mm_Drill1.0mm, RF_Custom:Pad_D1.5mm_Drill1.0mm, F.Cu at (121.9, 193.0)
- added REF**: Pad_D1.5mm_Drill1.0mm, RF_Custom:Pad_D1.5mm_Drill1.0mm, F.Cu at (144.8, 106.7)
- added REF**: Pad_D1.5mm_Drill1.0mm, RF_Custom:Pad_D1.5mm_Drill1.0mm, F.Cu at (137.2, 180.3)
- added REF**: Pad_D1.5mm_Drill1.0mm, RF_Custom:Pad_D1.5mm_Drill1.0mm, F.Cu at (142.2, 109.2)
- added REF**: Pad_D1.5mm_Drill1.0mm, RF_Custom:Pad_D1.5mm_Drill1.0mm, F.Cu at (127.0, 200.7)
- added REF**: Pad_D1.5mm_Drill1.0mm, RF_Custom:Pad_D1.5mm_Drill1.0mm, F.Cu at (139.7, 111.8)
- added REF**: Pad_D1.5mm_Drill1.0mm, RF_Custom:Pad_D1.5mm_Drill1.0mm, F.Cu at (137.2, 182.9)
- added REF**: Pad_D1.5mm_Drill1.0mm, RF_Custom:Pad_D1.5mm_Drill1.0mm, F.Cu at (114.3, 109.2)
- added REF**: Pad_D1.5mm_Drill1.0mm, RF_Custom:Pad_D1.5mm_Drill1.0mm, F.Cu at (127.0, 215.9)
- added REF**: Pad_D1.5mm_Drill1.0mm, RF_Custom:Pad_D1.5mm_Drill1.0mm, F.Cu at (121.9, 188.0)
- added REF**: Pad_D1.5mm_Drill1.0mm, RF_Custom:Pad_D1.5mm_Drill1.0mm, F.Cu at (124.5, 203.2)
- added REF**: Pad_D1.5mm_Drill1.0mm, RF_Custom:Pad_D1.5mm_Drill1.0mm, F.Cu at (137.2, 236.2)
- added REF**: Pad_D1.5mm_Drill1.0mm, RF_Custom:Pad_D1.5mm_Drill1.0mm, F.Cu at (119.4, 109.2)
- added REF**: Pad_D1.5mm_Drill1.0mm, RF_Custom:Pad_D1.5mm_Drill1.0mm, F.Cu at (137.2, 109.2)
- added REF**: Pad_D1.5mm_Drill1.0mm, RF_Custom:Pad_D1.5mm_Drill1.0mm, F.Cu at (134.6, 185.4)
- added REF**: Pad_D1.5mm_Drill1.0mm, RF_Custom:Pad_D1.5mm_Drill1.0mm, F.Cu at (121.9, 116.8)
- added REF**: Pad_D1.5mm_Drill1.0mm, RF_Custom:Pad_D1.5mm_Drill1.0mm, F.Cu at (129.5, 180.3)
- added REF**: Pad_D1.5mm_Drill1.0mm, RF_Custom:Pad_D1.5mm_Drill1.0mm, F.Cu at (121.9, 213.4)
- added REF**: Pad_D1.5mm_Drill1.0mm, RF_Custom:Pad_D1.5mm_Drill1.0mm, F.Cu at (132.1, 185.4)
- added REF**: Pad_D1.5mm_Drill1.0mm, RF_Custom:Pad_D1.5mm_Drill1.0mm, F.Cu at (129.5, 231.1)
- added REF**: Pad_D1.5mm_Drill1.0mm, RF_Custom:Pad_D1.5mm_Drill1.0mm, F.Cu at (129.5, 208.3)
- added REF**: Pad_D1.5mm_Drill1.0mm, RF_Custom:Pad_D1.5mm_Drill1.0mm, F.Cu at (137.2, 195.6)
- added REF**: Pad_D1.5mm_Drill1.0mm, RF_Custom:Pad_D1.5mm_Drill1.0mm, F.Cu at (129.5, 188.0)
- added REF**: Pad_D1.5mm_Drill1.0mm, RF_Custom:Pad_D1.5mm_Drill1.0mm, F.Cu at (111.8, 116.8)
- added REF**: Pad_D1.5mm_Drill1.0mm, RF_Custom:Pad_D1.5mm_Drill1.0mm, F.Cu at (129.4, 175.3)
- added REF**: Pad_D1.5mm_Drill1.0mm, RF_Custom:Pad_D1.5mm_Drill1.0mm, F.Cu at (121.8, 170.2)
- added REF**: Pad_D1.5mm_Drill1.0mm, RF_Custom:Pad_D1.5mm_Drill1.0mm, F.Cu at (134.6, 195.6)
- added REF**: Pad_D1.5mm_Drill1.0mm, RF_Custom:Pad_D1.5mm_Drill1.0mm, F.Cu at (116.8, 116.8)
- added REF**: Pad_D1.5mm_Drill1.0mm, RF_Custom:Pad_D1.5mm_Drill1.0mm, F.Cu at (137.1, 172.7)
- added REF**: Pad_D1.5mm_Drill1.0mm, RF_Custom:Pad_D1.5mm_Drill1.0mm, F.Cu at (139.7, 182.9)
- added REF**: Pad_D1.5mm_Drill1.0mm, RF_Custom:Pad_D1.5mm_Drill1.0mm, F.Cu at (124.5, 198.1)
- added REF**: Pad_D1.5mm_Drill1.0mm, RF_Custom:Pad_D1.5mm_Drill1.0mm, F.Cu at (127.0, 210.8)
- added REF**: Pad_D1.5mm_Drill1.0mm, RF_Custom:Pad_D1.5mm_Drill1.0mm, F.Cu at (134.6, 215.9)
- added REF**: Pad_D1.5mm_Drill1.0mm, RF_Custom:Pad_D1.5mm_Drill1.0mm, F.Cu at (121.8, 175.3)
- added REF**: Pad_D1.5mm_Drill1.0mm, RF_Custom:Pad_D1.5mm_Drill1.0mm, F.Cu at (127.0, 116.8)
- added REF**: Pad_D1.5mm_Drill1.0mm, RF_Custom:Pad_D1.5mm_Drill1.0mm, F.Cu at (142.2, 231.1)
- added REF**: Pad_D1.5mm_Drill1.0mm, RF_Custom:Pad_D1.5mm_Drill1.0mm, F.Cu at (124.5, 116.8)
- added REF**: Pad_D1.5mm_Drill1.0mm, RF_Custom:Pad_D1.5mm_Drill1.0mm, F.Cu at (139.7, 193.0)
- added REF**: Pad_D1.5mm_Drill1.0mm, RF_Custom:Pad_D1.5mm_Drill1.0mm, F.Cu at (111.8, 106.7)
- added REF**: Pad_D1.5mm_Drill1.0mm, RF_Custom:Pad_D1.5mm_Drill1.0mm, F.Cu at (132.0, 175.3)
- added REF**: Pad_D1.5mm_Drill1.0mm, RF_Custom:Pad_D1.5mm_Drill1.0mm, F.Cu at (134.6, 231.1)
- added REF**: Pad_D1.5mm_Drill1.0mm, RF_Custom:Pad_D1.5mm_Drill1.0mm, F.Cu at (137.1, 177.6)
- added REF**: Pad_D1.5mm_Drill1.0mm, RF_Custom:Pad_D1.5mm_Drill1.0mm, F.Cu at (139.6, 170.2)
- added REF**: Pad_D1.5mm_Drill1.0mm, RF_Custom:Pad_D1.5mm_Drill1.0mm, F.Cu at (134.6, 203.2)
- added REF**: Pad_D1.5mm_Drill1.0mm, RF_Custom:Pad_D1.5mm_Drill1.0mm, F.Cu at (149.9, 111.8)
- added REF**: Pad_D1.5mm_Drill1.0mm, RF_Custom:Pad_D1.5mm_Drill1.0mm, F.Cu at (134.6, 116.8)
- added REF**: Pad_D1.5mm_Drill1.0mm, RF_Custom:Pad_D1.5mm_Drill1.0mm, F.Cu at (124.5, 193.0)
- added REF**: Pad_D1.5mm_Drill1.0mm, RF_Custom:Pad_D1.5mm_Drill1.0mm, F.Cu at (109.2, 106.7)
- added REF**: Pad_D1.5mm_Drill1.0mm, RF_Custom:Pad_D1.5mm_Drill1.0mm, F.Cu at (147.3, 111.8)
- added REF**: Pad_D1.5mm_Drill1.0mm, RF_Custom:Pad_D1.5mm_Drill1.0mm, F.Cu at (127.0, 203.2)
- added REF**: Pad_D1.5mm_Drill1.0mm, RF_Custom:Pad_D1.5mm_Drill1.0mm, F.Cu at (127.0, 182.9)
- added REF**: Pad_D1.5mm_Drill1.0mm, RF_Custom:Pad_D1.5mm_Drill1.0mm, F.Cu at (121.9, 114.3)
- added REF**: Pad_D1.5mm_Drill1.0mm, RF_Custom:Pad_D1.5mm_Drill1.0mm, F.Cu at (127.0, 185.4)
- added REF**: Pad_D1.5mm_Drill1.0mm, RF_Custom:Pad_D1.5mm_Drill1.0mm, F.Cu at (132.1, 195.6)
- added REF**: Pad_D1.5mm_Drill1.0mm, RF_Custom:Pad_D1.5mm_Drill1.0mm, F.Cu at (121.9, 106.7)
- added REF**: Pad_D1.5mm_Drill1.0mm, RF_Custom:Pad_D1.5mm_Drill1.0mm, F.Cu at (124.5, 210.8)
- added REF**: Pad_D1.5mm_Drill1.0mm, RF_Custom:Pad_D1.5mm_Drill1.0mm, F.Cu at (127.0, 228.6)
- added REF**: Pad_D1.5mm_Drill1.0mm, RF_Custom:Pad_D1.5mm_Drill1.0mm, F.Cu at (124.5, 236.2)
- added REF**: Pad_D1.5mm_Drill1.0mm, RF_Custom:Pad_D1.5mm_Drill1.0mm, F.Cu at (127.0, 188.0)
- added REF**: Pad_D1.5mm_Drill1.0mm, RF_Custom:Pad_D1.5mm_Drill1.0mm, F.Cu at (121.9, 109.2)
- added REF**: Pad_D1.5mm_Drill1.0mm, RF_Custom:Pad_D1.5mm_Drill1.0mm, F.Cu at (134.6, 180.3)
- added REF**: Pad_D1.5mm_Drill1.0mm, RF_Custom:Pad_D1.5mm_Drill1.0mm, F.Cu at (132.0, 170.2)
- added REF**: Pad_D1.5mm_Drill1.0mm, RF_Custom:Pad_D1.5mm_Drill1.0mm, F.Cu at (139.7, 221.0)
- added REF**: Pad_D1.5mm_Drill1.0mm, RF_Custom:Pad_D1.5mm_Drill1.0mm, F.Cu at (137.2, 106.7)
- added REF**: Pad_D1.5mm_Drill1.0mm, RF_Custom:Pad_D1.5mm_Drill1.0mm, F.Cu at (139.7, 195.6)
- added REF**: Pad_D1.5mm_Drill1.0mm, RF_Custom:Pad_D1.5mm_Drill1.0mm, F.Cu at (127.0, 195.6)
- added REF**: Pad_D1.5mm_Drill1.0mm, RF_Custom:Pad_D1.5mm_Drill1.0mm, F.Cu at (124.5, 195.6)
- added REF**: Pad_D1.5mm_Drill1.0mm, RF_Custom:Pad_D1.5mm_Drill1.0mm, F.Cu at (139.6, 177.6)
- added REF**: Pad_D1.5mm_Drill1.0mm, RF_Custom:Pad_D1.5mm_Drill1.0mm, F.Cu at (119.4, 106.7)
- added REF**: Pad_D1.5mm_Drill1.0mm, RF_Custom:Pad_D1.5mm_Drill1.0mm, F.Cu at (124.5, 106.7)
- added REF**: Pad_D1.5mm_Drill1.0mm, RF_Custom:Pad_D1.5mm_Drill1.0mm, F.Cu at (114.3, 116.8)
- added REF**: Pad_D1.5mm_Drill1.0mm, RF_Custom:Pad_D1.5mm_Drill1.0mm, F.Cu at (127.0, 208.3)
- added REF**: Pad_D1.5mm_Drill1.0mm, RF_Custom:Pad_D1.5mm_Drill1.0mm, F.Cu at (139.7, 223.5)
- added REF**: Pad_D1.5mm_Drill1.0mm, RF_Custom:Pad_D1.5mm_Drill1.0mm, F.Cu at (127.0, 205.7)
- added REF**: Pad_D1.5mm_Drill1.0mm, RF_Custom:Pad_D1.5mm_Drill1.0mm, F.Cu at (134.5, 172.7)
- added REF**: Pad_D1.5mm_Drill1.0mm, RF_Custom:Pad_D1.5mm_Drill1.0mm, F.Cu at (137.2, 190.5)
- added REF**: Pad_D1.5mm_Drill1.0mm, RF_Custom:Pad_D1.5mm_Drill1.0mm, F.Cu at (124.5, 215.9)
- added REF**: Pad_D1.5mm_Drill1.0mm, RF_Custom:Pad_D1.5mm_Drill1.0mm, F.Cu at (121.9, 180.3)
- added REF**: Pad_D1.5mm_Drill1.0mm, RF_Custom:Pad_D1.5mm_Drill1.0mm, F.Cu at (139.7, 188.0)
- added REF**: Pad_D1.5mm_Drill1.0mm, RF_Custom:Pad_D1.5mm_Drill1.0mm, F.Cu at (129.5, 233.7)
- added REF**: Pad_D1.5mm_Drill1.0mm, RF_Custom:Pad_D1.5mm_Drill1.0mm, F.Cu at (134.6, 233.7)
- added REF**: Pad_D1.5mm_Drill1.0mm, RF_Custom:Pad_D1.5mm_Drill1.0mm, F.Cu at (129.4, 172.7)
- added REF**: Pad_D1.5mm_Drill1.0mm, RF_Custom:Pad_D1.5mm_Drill1.0mm, F.Cu at (134.6, 221.0)
- added REF**: Pad_D1.5mm_Drill1.0mm, RF_Custom:Pad_D1.5mm_Drill1.0mm, F.Cu at (139.6, 172.7)
- added REF**: Pad_D1.5mm_Drill1.0mm, RF_Custom:Pad_D1.5mm_Drill1.0mm, F.Cu at (132.1, 193.0)
- added REF**: Pad_D1.5mm_Drill1.0mm, RF_Custom:Pad_D1.5mm_Drill1.0mm, F.Cu at (124.5, 111.8)
- added REF**: Pad_D1.5mm_Drill1.0mm, RF_Custom:Pad_D1.5mm_Drill1.0mm, F.Cu at (132.1, 198.1)
- added REF**: Pad_D1.5mm_Drill1.0mm, RF_Custom:Pad_D1.5mm_Drill1.0mm, F.Cu at (137.2, 208.3)
- added REF**: Pad_D1.5mm_Drill1.0mm, RF_Custom:Pad_D1.5mm_Drill1.0mm, F.Cu at (127.0, 236.2)
- added REF**: Pad_D1.5mm_Drill1.0mm, RF_Custom:Pad_D1.5mm_Drill1.0mm, F.Cu at (132.1, 210.8)
- added REF**: Pad_D1.5mm_Drill1.0mm, RF_Custom:Pad_D1.5mm_Drill1.0mm, F.Cu at (139.7, 109.2)
- added REF**: Pad_D1.5mm_Drill1.0mm, RF_Custom:Pad_D1.5mm_Drill1.0mm, F.Cu at (137.2, 213.4)
- added REF**: Pad_D1.5mm_Drill1.0mm, RF_Custom:Pad_D1.5mm_Drill1.0mm, F.Cu at (144.8, 228.6)
- added REF**: Pad_D1.5mm_Drill1.0mm, RF_Custom:Pad_D1.5mm_Drill1.0mm, F.Cu at (124.5, 223.5)
- added REF**: Pad_D1.5mm_Drill1.0mm, RF_Custom:Pad_D1.5mm_Drill1.0mm, F.Cu at (139.7, 233.7)
- added REF**: Pad_D1.5mm_Drill1.0mm, RF_Custom:Pad_D1.5mm_Drill1.0mm, F.Cu at (142.2, 116.8)
- added REF**: Pad_D1.5mm_Drill1.0mm, RF_Custom:Pad_D1.5mm_Drill1.0mm, F.Cu at (134.6, 236.2)
- added REF**: Pad_D1.5mm_Drill1.0mm, RF_Custom:Pad_D1.5mm_Drill1.0mm, F.Cu at (134.5, 170.2)
- added REF**: Pad_D1.5mm_Drill1.0mm, RF_Custom:Pad_D1.5mm_Drill1.0mm, F.Cu at (124.5, 109.2)
- added REF**: Pad_D1.5mm_Drill1.0mm, RF_Custom:Pad_D1.5mm_Drill1.0mm, F.Cu at (142.2, 226.1)
- added REF**: Pad_D1.5mm_Drill1.0mm, RF_Custom:Pad_D1.5mm_Drill1.0mm, F.Cu at (127.0, 193.0)
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- renumbered C3 to C10, C4 to C14, C5 to C16, C8 to C18, C6 to C21, C10 to C23, C2 to C5, D6 to D10, D7 to D11, D8 to D12, D9 to D13, D10 to D14, D11 to D15, D12 to D16, D13 to D17, D14 to D18, D15 to D19, D16 to D20, D17 to D21, D18 to D22, D19 to D23, D20 to D24, D21 to D25, D22 to D26, D1 to D4, D2 to D5, D3 to D7, D4 to D8, D5 to D9, J2 to J1, J7 to J12, J8 to J13, J12 to J16, J13 to J17, J15 to J18, J3 to J2, J11 to J21, J9 to J22, J16 to J26, J17 to J27, J18 to J28, J19 to J29, J5 to J3, J4 to J5, J1 to J6, J6 to J8, R4 to R10, R6 to R11, R7 to R12, R8 to R16, R9 to R21, R10 to R22, R11 to R23, R12 to R24, R13 to R25, R14 to R26, R15 to R27, R16 to R28, R17 to R29, R18 to R30, R19 to R31, R20 to R32, R21 to R33, R22 to R34, R23 to R35, R24 to R36, R25 to R37, R26 to R38, R27 to R39, R28 to R40, R29 to R41, R30 to R42, R31 to R43, R32 to R44, R33 to R45, R34 to R46, R35 to R47, R36 to R48, R37 to R49, R38 to R50, R39 to R51, R40 to R52, R1 to R7, R3 to R9
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Connections:
- net /-5V renamed /-12V
- A1 pad 5V1: 5V -> /5V
- A1 pad 5V2: 5V -> /5V
- A1 pad 5V3: 5V -> /5V
- A1 pad 5V4: 5V -> /5V
- A1 pad A12: unconnected-(A1-PadA12) -> Net-(J24-Pin_1)
- A1 pad A13: unconnected-(A1-PadA13) -> Net-(J24-Pin_2)
- A1 pad A14: unconnected-(A1-PadA14) -> Net-(J24-Pin_3)
- A1 pad A15: unconnected-(A1-PadA15) -> Net-(J24-Pin_4)
- A1 pad A4: unconnected-(A1-PadA4) -> Net-(J23-Pin_1)
- A1 pad A5: unconnected-(A1-PadA5) -> Net-(J23-Pin_2)
- A1 pad A6: unconnected-(A1-PadA6) -> Net-(J23-Pin_3)
- A1 pad A7: unconnected-(A1-PadA7) -> Net-(J23-Pin_4)
- A1 pad D12: /START -> Net-(A1-PadD12)
- A1 pad D13: unconnected-(A1-PadD13) -> /D13
- A1 pad D14: RXD -> Net-(A1-D14/TX3)
- A1 pad D15: TXD -> Net-(A1-D15/RX3)
- A1 pad D16: RESET -> Net-(A1-D16/TX2)
- A1 pad D17: TX INHIBIT -> Net-(A1-D17/RX2)
- A1 pad D18: STBY 144 -> Net-(A1-D18/TX1)
- A1 pad D19: STBY 50 -> Net-(A1-D19/RX1)
- A1 pad D2: STBY HF -> Net-(A1-D2_INT0)
- A1 pad D20: SDA -> /SDA
- A1 pad D21: SCL -> /SCL
- A1 pad D22: /SEQ-A-RX -> /D22
- A1 pad D23: /SEQ-A-1 -> /D23
- A1 pad D24: /SEQ-A-2 -> /D24
- A1 pad D25: /SEQ-A-3 -> /D25
- A1 pad D26: /SEQ-A-TX -> /D26
- A1 pad D27: /SEQ-B-RX -> /D27
- A1 pad D28: /SEQ-B-1 -> /D28
- A1 pad D29: /SEQ-B-2 -> /D29
- A1 pad D3: STBY 430 -> Net-(A1-D3_INT1)
- A1 pad D30: /SEQ-B-3 -> /D30
- A1 pad D31: /SEQ-B-TX -> /D31
- A1 pad D32: unconnected-(A1-PadD32) -> /D32
- A1 pad D33: unconnected-(A1-PadD33) -> /D33
- A1 pad D34: unconnected-(A1-PadD34) -> /SEQ-A-RX
- A1 pad D35: unconnected-(A1-PadD35) -> /SEQ-A-1
- A1 pad D36: unconnected-(A1-PadD36) -> /SEQ-A-2
- A1 pad D37: unconnected-(A1-PadD37) -> /SEQ-A-3
- A1 pad D38: unconnected-(A1-PadD38) -> /SEQ-A-TX
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Routing:
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- added copper zone on B.Cu, net /PGND
- added copper zone on F.Cu, net /PGND
Other:
- board size 160.4 x 158.2 mm -> 214 x 204 mm
- board text added: "1 2 3 4 5"
- board text added: "13.8v 5v GND D13 D22 D23 D24 D25 D26 D27 D28 D29 D30 D31 D32 D33"
- board text added: "5 4 3 2 1"
- board text added: "50 144 HF 430 GND"
- board text added: "A12 A13 A14 A15"
- board text added: "A4 A5 A6 A7"
- board text added: "ALC"
- board text added: "ALC TRIM"
- board text added: "ANALOG"
- board text added: "ATU"
- board text added: "ATU FUSE 1A"
- board text added: "C A T"
- board text added: "EXT POWER"
- board text added: "G3ACE - Yaesu FT847 to Icom Tuner and 4 Band Sequencer Interface V1.1"
- board text added: "GND 13.8v 5v D13 D22 D23 D24 D25 D26 D27 D28 D29 D30 D31 D32 D33 GND"
- board text added: "GND 5V SCL SDA"
- board text added: "GND RADIO RX RADIO TX GND PC RX PC TX"
- board text added: "I 2 C"
- board text added: "I2C BUS"
- board text added: "KEY SRT 12V GND"
- board text added: "P13.8V"
- board text added: "PCTX PCRX GND RTX RRX GND"
- board text added: "PGND"
- board text added: "PGND P13.8V START KEY"
- board text added: "PROTOTYPE AREAS"
- board text added: "Pinout: C1 E1 C2 E2 C3 E3"
- board text added: "R13.8V LINK"
- board text added: "S P A R E"
- board text added: "SDA SCL 5V GND"
- board text added: "SERIAL/CAT"
- board text added: "SPARE"
- board text added: "TUNE STATUS"
- board text removed: "13.8V PGND KEY START"
- board text removed: "5V GND SDA SCL"
- board text removed: "ALC OUT"
- board text removed: "G3ACE - Yaesu FT847 to Icom Tuner and 4 Band Sequencer Interface V1.0"
- board text removed: "I2C"
- board text removed: "ICOM ATU"
- board text removed: "POWER"
- board text removed: "Pinout: E1 C1 E2 C2 E3 C3"
- board text removed: "SRT KEY GND 12V"
- board text removed: "TXGND LINK"

Commit message: Update schematic and PCB with ALC 10 turn pot
Parts:
- RV1: value 100K -> 47K; footprint Potentiometer_THT:Potentiometer_Runtron_RM-065_Vertical -> Potentiometer_THT:Potentiometer_Bourns_3296W_Vertical
- turned RV1 to -90 degrees
Routing:
- net /-4V: track 29.4 -> 34.4 mm
