File: kicad/yaesu_icom_atu_seq_v2/yaesu_icom_atu_seq_v2.kicad_pcb (KiCad board)
At the start: 2 copper layers, 214 x 204 mm, 506 parts, among them J1 STBY, J10 P13.8V, J11 SPARE, J12 STBY, J13 TUNER, J14 I2C, J15 SERIAL, J16 POWER, J17 Icom ATU, J18 ALC OUT, J19 SPARE, J2 TUNER, J20 RVLINK, J21 PGLINK, J22 PVLINK, J23 ANALOG, J24 ANALOG, J25 EXP, J26 SEQ A1-3, J27 SEQ B1-3, J28 SEQ C1-3, J29 SEQ D1-3, J3 I2C, J4 SERIAL, J5 POWER, J6 ICOM ATU, J7 SPARE, J8 ALC, J9 PGND, Q1 BC547, SW1 TUNE, U1 PC817, U2 L7805, U3 MAX202CPE, U4 PC817, U5 PC817, U6 PC817, U7 PC817

Commit message: add PCB production files
Parts:
- added C1: 100n, Capacitor_THT:C_Disc_D4.3mm_W1.9mm_P5.00mm, F.Cu at (142.6, 87.6)
- renumbered C9 to C10, C10 to C11, C11 to C12, C12 to C13, C13 to C14, C14 to C15, C15 to C16, C16 to C17, C17 to C18, C18 to C19, C1 to C2, C19 to C20, C20 to C21, C21 to C22, C22 to C23, C23 to C24, C24 to C25, C25 to C26, C26 to C27, C27 to C28, C28 to C29, C2 to C3, C29 to C30, C30 to C31, C31 to C32, C32 to C33, C33 to C34, C34 to C35, C35 to C36, C36 to C37, C3 to C4, C4 to C5, C5 to C6, C6 to C7, C7 to C8, C8 to C9
Routing:
- net /5V: track 478.0 -> 481.1 mm
- net GND: vias 168 -> 169

Commit message: update schematic and pcb with new 9V supply for thr ALC circuit, re-publish gerbers
Parts:
- added C38: 47u, Capacitor_THT:CP_Radial_D5.0mm_P2.50mm, F.Cu at (261.6, 149.9)
- added C39: 100n, Capacitor_THT:C_Disc_D4.3mm_W1.9mm_P5.00mm, F.Cu at (261.6, 144.8)
- added D40: 1N4001, Diode_THT:D_DO-35_SOD27_P7.62mm_Horizontal, F.Cu at (284.5, 141.0)
- added J30: 9V, Connector_PinHeader_2.54mm:PinHeader_2x02_P2.54mm_Vertical, F.Cu at (254.0, 149.9)
- added REF**: PinHeader_1x08_P2.54mm_Vertical, Connector_PinHeader_2.54mm:PinHeader_1x08_P2.54mm_Vertical, F.Cu at (250.2, 98.0)
- added REF**: PinHeader_1x08_P2.54mm_Vertical, Connector_PinHeader_2.54mm:PinHeader_1x08_P2.54mm_Vertical, F.Cu at (201.9, 115.8)
- added REF**: PinHeader_1x08_P2.54mm_Vertical, Connector_PinHeader_2.54mm:PinHeader_1x08_P2.54mm_Vertical, F.Cu at (201.9, 93.0)
- added REF**: PinHeader_1x08_P2.54mm_Vertical, Connector_PinHeader_2.54mm:PinHeader_1x08_P2.54mm_Vertical, F.Cu at (250.2, 120.9)
- added REF**: PinHeader_2x18_P2.54mm_Vertical, Connector_PinHeader_2.54mm:PinHeader_2x18_P2.54mm_Vertical, F.Cu at (245.1, 141.2)
- added REF**: PinHeader_1x08_P2.54mm_Vertical, Connector_PinHeader_2.54mm:PinHeader_1x08_P2.54mm_Vertical, F.Cu at (250.2, 75.2)
- added REF**: PinHeader_1x10_P2.54mm_Vertical, Connector_PinHeader_2.54mm:PinHeader_1x10_P2.54mm_Vertical, F.Cu at (201.9, 66.0)
- added U8: L78L09, Package_TO_SOT_THT:TO-92_Inline, F.Cu at (265.4, 146.1)
- BZ1: footprint Buzzer_Beeper:Buzzer_TDK_PS1240P02BT_D12.2mm_H6.5mm -> Buzzer_Beeper:Buzzer_12x9.5RM7.6
- C19, C2: value 100u -> 47u
- F1: footprint Fuse:Fuse_Blade_ATO_directSolder -> Custom:Fuse_Blade_ATO_directSolder (longer holes)
- R1, R14, R2, R20, R3, R4: value 1K -> 470R
- R10, R11, R12, R9: value 1K -> 47K
- R17: value 1K -> 10K
- R19, R21, R22, R23, R24, R25, R26, R27, R28, R29, R30, R31, R32, R33, R34, R35, R36, R37, R38, R39, R40: value 1K -> 3K9
- R41, R42, R43, R44, R45, R46, R47, R48, R49, R50, R51, R52, R7: value 1K -> 1K8
- R5: value 1K -> 680R
- R53, R54, R55, R56, R57, R58, R59, R6, R60, R61, R62, R63, R64: value 1K -> 100R
- moved R14 11.4 mm to (266.7, 139.7), turned to 90 degrees
- moved C19 9.15 mm to (271.8, 135.9), turned to -90 degrees
- moved C17 7.70 mm to (276.9, 135.9), turned to -90 degrees
- moved J22 3.89 mm to (292.6, 133.3), turned to 90 degrees
- moved C2 2.92 mm to (292.1, 141.6)
- moved C6 1.27 mm to (288.3, 141.7)
Connections:
- net /-12V renamed /-7.5V
- net /-4V renamed /-4.6V
- C2 pad 1: /13.8V -> Net-(D40-K)
- C6 pad 1: /13.8V -> Net-(D40-K)
- R14 pad 1: /13.8V -> /9V
- U2 pad 1: /13.8V -> Net-(D40-K)
Routing:
- net Net-(D40-K): track 0.00 -> 30.7 mm
- net /9V: track 0.00 -> 29.7 mm
- net /13.8V: track 213.2 -> 198.4 mm
- net GND: track 173.1 -> 183.3 mm, vias 169 -> 170
- net /P13.8V: track 169.5 -> 164.3 mm
- net Net-(Q1-C): track 11.5 -> 16.6 mm
- net /5V: track 481.1 -> 484.8 mm
Other:
- board text added: "9V"
- board text added: "G3ACE - Yaesu FT847 to Icom Tuner and 4 Band Sequencer Interface V1.2"
- board text removed: "G3ACE - Yaesu FT847 to Icom Tuner and 4 Band Sequencer Interface V1.1"
