File: kicad/yaesu_icom_atu_seq_v2/yaesu_icom_atu_seq_v2.kicad_sch (KiCad schematic)
At the start: 191 parts, among them J1 STBY, J10 P13.8V, J11 SPARE, J12 STBY, J13 TUNER, J14 I2C, J15 SERIAL, J16 POWER, J17 Icom ATU, J18 ALC OUT, J19 SPARE, J2 TUNER, J20 RVLINK, J21 PGLINK, J22 PVLINK, J23 ANALOG, J24 ANALOG, J25 EXP, J26 SEQ A1-3, J27 SEQ B1-3, J28 SEQ C1-3, J29 SEQ D1-3, J3 I2C, J4 SERIAL, J5 POWER, J6 ICOM ATU, J7 SPARE, J8 ALC, J9 PGND, Q1 BC547, SW1 TUNE, U1 PC817, U2 L7805, U3 MAX202CPE, U4 PC817, U5 PC817, U6 PC817, U7 PC817

Commit message: add PCB production files
Parts:
- added C1: 100n, Capacitor_THT:C_Disc_D4.3mm_W1.9mm_P5.00mm, symbol Device:C_Small
- R1, R2, R20, R3, R4: value 1K -> 470R
- R10, R11, R12, R9: value 1K -> 47K
- R17: value 1K -> 10K
- R19, R21, R22, R23, R24, R25, R26, R27, R28, R29, R30, R31, R32, R33, R34, R35, R36, R37, R38, R39, R40: value 1K -> 4K7
- R41, R42, R43, R44, R45, R46, R47, R48, R49, R50, R51, R52, R7: value 1K -> 1K8
- R5: value 1K -> 680R
- R53, R54, R55, R56, R57, R58, R59, R6, R60, R61, R62, R63, R64: value 1K -> 100R
- renumbered C9 to C10, C10 to C11, C11 to C12, C12 to C13, C13 to C14, C14 to C15, C15 to C16, C16 to C17, C17 to C18, C18 to C19, C1 to C2, C19 to C20, C20 to C21, C21 to C22, C22 to C23, C23 to C24, C24 to C25, C25 to C26, C26 to C27, C27 to C28, C28 to C29, C2 to C3, C29 to C30, C30 to C31, C31 to C32, C32 to C33, C33 to C34, C34 to C35, C35 to C36, C36 to C37, C3 to C4, C4 to C5, C5 to C6, C6 to C7, C7 to C8, C8 to C9
Connections:
- net 5V: now also C1.1
- net GND: now also C1.2

Commit message: update schematic and pcb with new 9V supply for thr ALC circuit, re-publish gerbers
Parts:
- added C38: 47u, Capacitor_THT:CP_Radial_D5.0mm_P2.50mm, symbol Device:C_Polarized_Small
- added C39: 100n, Capacitor_THT:C_Disc_D4.3mm_W1.9mm_P5.00mm, symbol Device:C_Small
- added D40: 1N4001, Diode_THT:D_DO-35_SOD27_P7.62mm_Horizontal, symbol Diode:1N4148
- added J30: 9V, Connector_PinHeader_2.54mm:PinHeader_2x02_P2.54mm_Vertical, symbol Connector_Generic:Conn_02x02_Counter_Clockwise
- added U8: L78L09, Package_TO_SOT_THT:TO-92_Inline, symbol Regulator_Linear:L78L09_TO92
- BZ1: footprint Buzzer_Beeper:Buzzer_TDK_PS1240P02BT_D12.2mm_H6.5mm -> Buzzer_Beeper:Buzzer_12x9.5RM7.6
- C19, C2: value 100u -> 47u
- F1: footprint Fuse:Fuse_Blade_ATO_directSolder -> Custom:Fuse_Blade_ATO_directSolder (longer holes)
- R14: value 1K -> 470R
- R19, R21, R22, R23, R24, R25, R26, R27, R28, R29, R30, R31, R32, R33, R34, R35, R36, R37, R38, R39, R40: value 4K7 -> 3K9
Connections:
- net 13.8V: now also D40.2 (A); no longer C2.1, C6.1, R14.1, U2.1 (IN)
- net GND: now also C38.2, C39.2, U8.2 (GND)
- net -12V renamed -7.5V
- net -4V renamed -4.6V
- new net: C2.1, C6.1, D40.1 (K), U2.1 (IN), U8.3 (VI)
- new net 9V: C38.1, C39.1, J30.1 (Pin_1), J30.2 (Pin_2), J30.3 (Pin_3), J30.4 (Pin_4), R14.1, U8.1 (VO)
Other:
- title: (none) -> G3ACE Yaesu FT-847 to Icom ATU and 4 Band Sequencer v1.2
- moved on the sheet: C17, C19, C2, C6, E1, J11, J18, J19, J7, J8, PR1, PR2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
